File: 03_hw_design/02_schematic_and_bom/01_Schematics_BOM/LLC_DCDC_V5_Modifications/GateDrivers.kicad_sch (KiCad schematic)
At the start: 39 parts, among them IC1 NCP43080DDR2G, IC7 NCP43080DDR2G, J2 jumper_02x03, J3 jumper_02x03, J4 jumper_02x03, J5 jumper_02x03, U2 UCC21520Q

Commit message: photos
Changed lines of the file:
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@@
 	(title_block
 		(title "LLC 400V/48V 1200W 100kHz")
-		(date "2025-10-14")
-		(rev "5")
+		(date "2026-02-01")
+		(rev "6")
 		(company "Abdelaziz BOUZIANI")
 	)
@@
 			)
 		)
-		(property "Description" "11.5k 1% 1/4W 1206"
+		(property "Description" "203 20k"
 			(at 66.04 40.6399 0)
 			(effects
@@
 			)
 		)
-		(property "Description" "11.5k 1% 1/4W 1206"
+		(property "Description" "203 20k"
 			(at 196.85 40.6399 0)
 			(effects
