File: 03_hw_design/02_schematic_and_bom/01_Schematics_BOM/LLC_DCDC_V5_Modifications/MUC_AND_OTHERS.kicad_sch (KiCad schematic)
At the start: 26 parts, among them IC10 ISO7741BDWR, IC6 SN74HC74DRG4, J1 Conn_02x03, J8 jumper_02x03, U1 stm32F103C8T6-CH340

Commit message: photos
Connections:
- net DisableHpVout: now reaches U1.14 (b11)
Other:
- note removed: "| Channel | Main Pin | Complementary Pin | | CH1 | PA8 | PB13 | | CH2 | PA9 | PB14 | | CH3 | PA10 | PB15 |"
Changed lines of the file:
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@@
 	(title_block
 		(title "LLC 400V/48V 1200W 100kHz")
-		(date "2025-10-14")
-		(rev "5")
+		(date "2026-02-01")
+		(rev "6")
 		(company "Abdelaziz BOUZIANI")
 	)
@@
 		)
 	)
-	(text "| Channel | Main Pin | Complementary Pin |\n| CH1     | PA8      | PB13              |\n| CH2     | PA9      | PB14              |\n| CH3     | PA10     | PB15              |"
-		(exclude_from_sim no)
-		(at 209.804 89.916 0)
-		(effects
-			(font
-				(size 1.27 1.27)
-			)
-			(justify left)
-		)
-	)
 	(text "open= Enable\n"
 		(exclude_from_sim no)
@@
 	(wire
 		(pts
+			(xy 97.79 104.14) (xy 97.79 109.22)
+		)
+		(stroke
+			(width 0)
+			(type default)
+		)
+	)
+	(wire
+		(pts
 			(xy 196.85 26.67) (xy 193.04 26.67)
 		)
@@
 	(wire
 		(pts
+			(xy 97.79 109.22) (xy 100.33 109.22)
+		)
+		(stroke
+			(width 0)
+			(type default)
+		)
+	)
+	(wire
+		(pts
 			(xy 73.66 41.91) (xy 76.2 41.91)
 		)
@@
 	(wire
 		(pts
+			(xy 96.52 104.14) (xy 97.79 104.14)
+		)
+		(stroke
+			(width 0)
+			(type default)
+		)
+	)
+	(wire
+		(pts
 			(xy 195.58 30.48) (xy 195.58 46.99)
 		)
@@
 			(effects
 				(font
+					(size 1.27 1.27)
+				)
+				(justify right)
+				(hide yes)
+			)
+		)
+	)
+	(global_label "DisableHpVout"
+		(shape input)
+		(at 96.52 104.14 180)
+		(fields_autoplaced yes)
+		(effects
+			(font
+				(size 1.27 1.27)
+			)
+			(justify right)
+		)
+		(property "Intersheetrefs" "${INTERSHEET_REFS}"
+			(at 79.9883 104.14 0)
+			(effects
+				(font
