File: 03_hw_design/02_schematic_and_bom/01_Schematics_BOM/LLC_DCDC_V5_Modifications/Power_Supplies.kicad_sch (KiCad schematic)
At the start: 49 parts, among them IC12 AZ1117CH2-3.3TRG1, IC13 LM4040AIM3-2.0, IC3 LM2575-3.3WU-TR, IC4 LM2575HVS-12_NOPB, J7 Conn_02x02_Odd_Even, Q5 DPC817S-B-TR, Q7 BCP5616H6327XTSA1, T2 Transformer_1P_1S

Commit message: draft push
Parts:
- added U3: TNY264G, Package_DIP:PowerIntegrations_SMD-8B, symbol Regulator_Switching:TNY264G
Connections:
- new net: U3.2 (S), U3.3 (S), U3.7 (S), U3.8 (S)
Other:
- note added: "100nF (of flyback charger, i measure it, 5.877v measurement)"
- note added: "TBC"
- note added: "TNY-264"
Changed lines of the file:
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@@
 		)
 	)
+	(text "TNY-264\n"
+		(exclude_from_sim no)
+		(at 56.642 78.486 0)
+		(effects
+			(font
+				(size 1.27 1.27)
+				(color 255 0 0 1)
+			)
+		)
+	)
+	(text "100nF (of flyback charger, i measure it, 5.877v measurement)\n"
+		(exclude_from_sim no)
+		(at 28.956 101.854 0)
+		(effects
+			(font
+				(size 1.27 1.27)
+				(color 255 0 0 1)
+			)
+		)
+	)
 	(text "https://www.power.com/products/tinyswitch/tinyswitch-iii/tny280p"
 		(exclude_from_sim no)
@@
 		)
 	)
+	(text "TBC"
+		(exclude_from_sim no)
+		(at 161.798 65.532 0)
+		(effects
+			(font
+				(size 1.27 1.27)
+				(color 255 0 0 1)
+			)
+		)
+	)
 	(text "Ref generator"
 		(exclude_from_sim no)
@@
 					(unit 1)
 				)
+			)
+		)
+	)
+	(symbol
+		(lib_id "Regulator_Switching:TNY264G")
+		(at 69.85 111.76 0)
+		(unit 1)
+		(exclude_from_sim no)
+		(in_bom yes)
+		(on_board yes)
+		(dnp no)
+		(fields_autoplaced yes)
+		(property "Reference" "U3"
+			(at 60.96 110.4899 0)
+			(effects
+				(font
+					(size 1.27 1.27)
+				)
+				(justify right)
+			)
+		)
+		(property "Value" "TNY264G"
+			(at 60.96 113.0299 0)
+			(effects
+				(font
+					(size 1.27 1.27)
+				)
+				(justify right)
+			)
+		)
+		(property "Footprint" "Package_DIP:PowerIntegrations_SMD-8B"
+			(at 69.85 111.76 0)
+			(effects
+				(font
+					(size 1.27 1.27)
+					(italic yes)
+				)
+				(hide yes)
+			)
+		)
+		(property "Datasheet" "http://www.powerint.com/sites/default/files/product-docs/tny263_268.pdf"
+			(at 69.85 111.76 0)
+			(effects
+				(font
+					(size 1.27 1.27)
+				)
+				(hide yes)
+			)
+		)
+		(property "Description" "TinySwitch-II Family, 6W Output Power, SMD-8B"
+			(at 69.85 111.76 0)
+			(effects
+				(font
+					(size 1.27 1.27)
+				)
+				(hide yes)
+			)
+		)
+		(pin "1"
+		)
+		(pin "7"
+		)
+		(pin "3"
+		)
+		(pin "8"
+		)
+		(pin "5"
+		)
+		(pin "4"
+		)
+		(pin "2"
+		)
+		(instances
+			(project ""
+				(path "/856dbdf2-f84a-4a26-871a-e6caa4757467/e6ae4412-3899-497a-ad4e-ef9e3f773d29"
+					(reference "U3")
+					(unit 1)
+				)

Commit message: push draft 12/02/2026
Parts:
- removed D2: US1J, Diode_SMD:D_SMA, symbol Diode:US1J
- removed D4: MBRS340T3G, MBRS340T3G:DIOM8059X261N, symbol MBRS340T3G:MBRS340T3G
- removed PS1: TNY280GN-TL, TNY280GN-TL:TNY280GNTL, symbol TNY280GN-TL:TNY280GN-TL
- removed Z1: BZT52C11-7-F, BZT52C11-7-F:SOD3716X145N, symbol BZT52C11-7-F:BZT52C11-7-F
- added D4: SB2100, symbol Device:D_Schottky
- added D5: US2MA, Diode_SMD:D_SMA, symbol Diode:US2MA
- added Z1: LLZ11, symbol Device:D_Zener
- Q5: value DPC817S-B-TR -> 817B
- T2: value Transformer_1P_1S -> ELP22/6/16 & I22/2.5/16 N87; Field5 NoAirGap -> B66285G0000X187 (ELP core) B66285K0000X187 (I core)
Connections:
- net +12drvPrim: now also D4.1 (K), Z1.1 (K)
- net GND_ISO: now also U3.2 (S), U3.3 (S), U3.7 (S), U3.8 (S)
- net at R12.1: now also Z1.2 (A)
- net at T2.4 (SB), TP22.1: now also D4.2 (A)
- net at T2.2 (AB), TP16.1: now also U3.5 (D), D5.2 (A)
- net at C23.2, R5.2, TP13.1: now also D5.1 (K)
- net at U3.1 (BP): now also C1.1
- net at U3.4 (EN/UV): now also Q5.4 (C), TP15.1
Other:
- note added: "FlyBack 400V/12V"
- note removed: "FlyBack 400/12/12"
- note removed: "TBC"
- note removed: "TNY-264"
- moved on the sheet: C1, C23, C46, C58, R5, TP13, TP16, TP22, U3
