File: 03_hw_design/02_schematic_and_bom/01_Schematics_BOM/LLC_DCDC_V5_Modifications/Power_components.kicad_sch (KiCad schematic)
At the start: 31 parts, among them Q1 IPW60R037CM8XKSA1, Q2 IPW60R037CM8XKSA1, Q3 FDH055N15A, Q4 FDH055N15A, T3 B66297K0000X197,B66297G0000X1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

Commit message: Lr Lm caract
Parts:
- Q1, Q2: value IPW60R037CM8XKSA1 -> IPW60R037P7; Height 5.21 -> (none); Manufacturer_Part_Number IPW60R037CM8XKSA1 -> (none); Mouser Part Number 726-IPW60R037CM8XKSA -> (none); Mouser Price/Stock https://www.mouser.co.uk/ProductDetail/Infineon-Technologie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 -> (none)
- Q3, Q4: value FDH055N15A -> IRFP4568PBF; Manufacturer_Name onsemi -> (none); Manufacturer_Part_Number FDH055N15A -> (none); Mouser Part Number 512-FDH055N15A -> (none); Mouser Price/Stock https://www.mouser.co.uk/ProductDetail/onsemi-Fairchild/FDH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 -> (none)
