File: 03_hw_design/02_schematic_and_bom/01_Schematics_BOM/LLC_DCDC_V5_Modifications/Sensors.kicad_sch (KiCad schematic)
At the start: 33 parts, among them IC5 SI8932B-IS, IC8 TMCS1107A1UQDRQ1, IC9 ACS70331EOLCTR-005U3, U9 TLV9024QDRQ1

Commit message: photos
Connections:
- net DisableHpVout: now reaches RV2.2, U9.6 (-)
Changed lines of the file:
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@@
 	(title_block
 		(title "LLC 400V/48V 1200W 100kHz")
-		(date "2025-10-14")
-		(rev "5")
+		(date "2026-02-01")
+		(rev "6")
 		(company "Abdelaziz BOUZIANI")
 	)
@@
 	)
 	(junction
+		(at 233.68 71.12)
+		(diameter 0)
+		(color 0 0 0 0)
+	)
+	(junction
 		(at 59.69 173.99)
 		(diameter 0)
@@
 	(wire
 		(pts
+			(xy 226.06 71.12) (xy 233.68 71.12)
+		)
+		(stroke
+			(width 0)
+			(type default)
+		)
+	)
+	(wire
+		(pts
 			(xy 233.68 107.95) (xy 229.87 107.95)
 		)
@@
 				(hide yes)
 			)
+		)
+	)
+	(global_label "DisableHpVout"
+		(shape input)
+		(at 226.06 71.12 180)
+		(fields_autoplaced yes)
+		(effects
+			(font
+				(size 1.27 1.27)
+			)
+			(justify right)
+		)
+		(property "Intersheetrefs" "${INTERSHEET_REFS}"
+			(at 209.5283 71.12 0)
+			(effects
+				(font
+					(size 1.27 1.27)
+				)
+				(justify right)
+				(hide yes)
+			)
